Commit message: Modifications to make things work with real hardware

File: ros2_control_demo_description/diffbot/urdf/diffbot_description.urdf.xacro (robot description, xacro)
@@ -43,5 +43,5 @@
       <origin xyz="0 -${base_width/2} ${z_offset}" rpy="0 0 0"/>
       <axis xyz="0 1 0"/>
-      <dynamics damping="0.2"/>
+      <dynamics damping="0.0"/>
       <limit effort="100" velocity="1.0"/>
     </joint>
@@ -73,7 +73,7 @@
       <parent link="${prefix}base_link"/>
       <child link="${prefix}right_wheel"/>
-      <origin xyz="0 ${base_width/2} ${z_offset}" rpy="0 0 0"/>
+      <origin xyz="0 ${base_width/2} ${z_offset}" rpy="0 0 ${PI}"/>
       <axis xyz="0 1 0"/>
-      <dynamics damping="0.2"/>
+      <dynamics damping="0.0"/>
       <limit effort="100" velocity="1.0"/>
     </joint>
